File: giulia.sch (KiCad schematic (older format))
At the start: 1 part

Commit message: basic MCU wiring
Parts:
- added C1, C2: 22p, symbol Device:C_Small
- added C3: 10u, symbol Device:CP_Small
- added C4, C5: 100n, symbol Device:C_Small
- added R1: 10k, symbol Device:R_Small
- added SW1: RESET, symbol Switch:SW_Push
- added Y1: 16 MHz, symbol Device:Crystal_Small
- gave numbers to parts that had none: 1
Connections:
- net +5V: now reaches U1.10 (VCC)
- net +5V: now also U1.30 (AVCC), C3.1, C4.1, C5.1, R1.1
- net GND: now reaches U1.11 (GND), U1.31 (GND)
- net GND: now also C1.2, C2.2, C3.2, C4.2, C5.2, SW1.1
- net at U1.12 (XTAL2): now also C2.1, Y1.2
- net at U1.13 (XTAL1): now also C1.1, Y1.1
- net at U1.9 (~RESET): now also R1.2, SW1.2
Other:
- moved on the sheet: U1
Changed lines of the file:
@@
 $EndDescr
 $Comp
-L MCU_Microchip_ATmega:ATmega32A-PU U?
+L MCU_Microchip_ATmega:ATmega32A-PU U1
 U 1 1 6106E53B
-P 1500 3400
-F 0 "U?" H 1500 1311 50  0000 C CNN
-F 1 "ATmega32A-PU" H 1500 1220 50  0000 C CNN
-F 2 "Package_DIP:DIP-40_W15.24mm" H 1500 3400 50  0001 C CIN
-F 3 "http://ww1.microchip.com/downloads/en/DeviceDoc/atmel-8155-8-bit-microcontroller-avr-atmega32a_datasheet.pdf" H 1500 3400 50  0001 C CNN
-	1    1500 3400
-	1    0    0    -1
-$EndComp
+P 5600 3750
+F 0 "U1" H 5500 3800 50  0000 C CNN
+F 1 "ATmega32A-PU" H 5500 3700 50  0000 C CNN
+F 2 "Package_DIP:DIP-40_W15.24mm" H 5600 3750 50  0001 C CIN
+F 3 "http://ww1.microchip.com/downloads/en/DeviceDoc/atmel-8155-8-bit-microcontroller-avr-atmega32a_datasheet.pdf" H 5600 3750 50  0001 C CNN
+	1    5600 3750
+	1    0    0    -1
+$EndComp
+$Comp
+L power:+5V #PWR?
+U 1 1 6107440A
+P 5600 1550
+F 0 "#PWR?" H 5600 1400 50  0001 C CNN
+F 1 "+5V" H 5615 1723 50  0000 C CNN
+F 2 "" H 5600 1550 50  0001 C CNN
+F 3 "" H 5600 1550 50  0001 C CNN
+	1    5600 1550
+	1    0    0    -1
+$EndComp
+Wire Wire Line
+	5600 1550 5600 1650
+Wire Wire Line
+	5700 1750 5700 1650
+Wire Wire Line
+	5700 1650 5600 1650
+Connection ~ 5600 1650
+Wire Wire Line
+	5600 1650 5600 1750
+$Comp
+L power:GND #PWR?
+U 1 1 610754C4
+P 5600 5850
+F 0 "#PWR?" H 5600 5600 50  0001 C CNN
+F 1 "GND" H 5605 5677 50  0000 C CNN
+F 2 "" H 5600 5850 50  0001 C CNN
+F 3 "" H 5600 5850 50  0001 C CNN
+	1    5600 5850
+	1    0    0    -1
+$EndComp
+$Comp
+L Device:C_Small C2
+U 1 1 6108361C
+P 4550 2650
+F 0 "C2" H 4650 2700 50  0000 L CNN
+F 1 "22p" H 4650 2600 50  0000 L CNN
+F 2 "" H 4550 2650 50  0001 C CNN
+F 3 "~" H 4550 2650 50  0001 C CNN
+	1    4550 2650
+	1    0    0    -1
+$EndComp
+$Comp
+L Device:C_Small C1
+U 1 1 61085D6B
+P 4350 2650
+F 0 "C1" H 4150 2700 50  0000 L CNN
+F 1 "22p" H 4150 2600 50  0000 L CNN
+F 2 "" H 4350 2650 50  0001 C CNN
+F 3 "~" H 4350 2650 50  0001 C CNN
+	1    4350 2650
+	1    0    0    -1
+$EndComp
+$Comp
+L power:GND #PWR?
+U 1 1 610873C2
+P 4550 2800
+F 0 "#PWR?" H 4550 2550 50  0001 C CNN
+F 1 "GND" H 4555 2627 50  0000 C CNN
+F 2 "" H 4550 2800 50  0001 C CNN
+F 3 "" H 4550 2800 50  0001 C CNN
+	1    4550 2800
+	1    0    0    -1
+$EndComp
+$Comp
+L Device:Crystal_Small Y1
+U 1 1 610C25E9
+P 4550 2350
+F 0 "Y1" V 4504 2438 50  0000 L CNN
+F 1 "16 MHz" V 4595 2438 50  0000 L CNN
+F 2 "" H 4550 2350 50  0001 C CNN
+F 3 "~" H 4550 2350 50  0001 C CNN
+	1    4550 2350
+	0    1    1    0
+$EndComp
+Wire Wire Line
+	5000 2250 4550 2250
+Wire Wire Line
+	5000 2450 4550 2450
+Wire Wire Line
+	4550 2250 4350 2250
+Wire Wire Line
+	4350 2250 4350 2550
+Connection ~ 4550 2250
+Wire Wire Line
+	4550 2550 4550 2450
+Connection ~ 4550 2450
+Wire Wire Line
+	4550 2750 4550 2800
+Wire Wire Line
+	4350 2750 4550 2750
+Connection ~ 4550 2750
+Wire Wire Line
+	5600 5850 5600 5750
+$Comp
+L power:+5V #PWR?
+U 1 1 610DE068
+P 4400 4950
+F 0 "#PWR?" H 4400 4800 50  0001 C CNN
+F 1 "+5V" H 4415 5123 50  0000 C CNN
+F 2 "" H 4400 4950 50  0001 C CNN
+F 3 "" H 4400 4950 50  0001 C CNN
+	1    4400 4950
+	1    0    0    -1
+$EndComp
+$Comp
+L Device:C_Small C4
+U 1 1 610DF006
+P 4400 5200
+F 0 "C4" H 4450 5350 50  0000 L CNN
+F 1 "100n" H 4450 5050 50  0000 L CNN
+F 2 "" H 4400 5200 50  0001 C CNN
+F 3 "~" H 4400 5200 50  0001 C CNN
+	1    4400 5200
+	1    0    0    -1
+$EndComp
+$Comp
+L Device:C_Small C5
+U 1 1 610E006A
+P 4550 5200
+F 0 "C5" H 4642 5246 50  0000 L CNN
+F 1 "100n" H 4642 5155 50  0000 L CNN
+F 2 "" H 4550 5200 50  0001 C CNN
+F 3 "~" H 4550 5200 50  0001 C CNN
+	1    4550 5200
+	1    0    0    -1
+$EndComp
+Wire Wire Line
+	4550 5100 4400 5100
+Connection ~ 4400 5100
+Wire Wire Line
+	4550 5300 4400 5300
+$Comp
+L Device:CP_Small C3
+U 1 1 610E14C2
+P 4250 5200
+F 0 "C3" H 4050 5250 50  0000 L CNN
+F 1 "10u" H 4050 5150 50  0000 L CNN
+F 2 "" H 4250 5200 50  0001 C CNN
+F 3 "~" H 4250 5200 50  0001 C CNN
+	1    4250 5200
+	1    0    0    -1
+$EndComp
+Wire Wire Line
+	4250 5100 4400 5100
+Wire Wire Line
+	4250 5300 4400 5300
+Connection ~ 4400 5300
+$Comp
+L power:GND #PWR?
+U 1 1 610E3173
+P 4400 5450
+F 0 "#PWR?" H 4400 5200 50  0001 C CNN
+F 1 "GND" H 4405 5277 50  0000 C CNN
+F 2 "" H 4400 5450 50  0001 C CNN
+F 3 "" H 4400 5450 50  0001 C CNN
+	1    4400 5450
+	1    0    0    -1
+$EndComp
+Wire Wire Line
+	4400 5450 4400 5300
+Wire Wire Line
+	4400 5100 4400 4950
+$Comp
+L Switch:SW_Push SW1
+U 1 1 610E88B8
+P 4600 2050
+F 0 "SW1" H 4600 2335 50  0000 C CNN
+F 1 "RESET" H 4600 2244 50  0000 C CNN
+F 2 "" H 4600 2250 50  0001 C CNN
+F 3 "~" H 4600 2250 50  0001 C CNN
+	1    4600 2050
+	1    0    0    -1
+$EndComp
+$Comp
+L power:GND #PWR?
+U 1 1 610E92D6
+P 4150 2050
+F 0 "#PWR?" H 4150 1800 50  0001 C CNN
+F 1 "GND" H 4155 1877 50  0000 C CNN
+F 2 "" H 4150 2050 50  0001 C CNN
+F 3 "" H 4150 2050 50  0001 C CNN
+	1    4150 2050
+	1    0    0    -1
+$EndComp
+Wire Wire Line
+	4150 2050 4400 2050
+$Comp
+L Device:R_Small R1
+U 1 1 610EA94C
+P 4900 1650
+F 0 "R1" H 4959 1696 50  0000 L CNN
+F 1 "10k" H 4959 1605 50  0000 L CNN
+F 2 "" H 4900 1650 50  0001 C CNN
+F 3 "~" H 4900 1650 50  0001 C CNN
+	1    4900 1650
+	1    0    0    -1
+$EndComp
+$Comp
+L power:+5V #PWR?
+U 1 1 610EB5A6
+P 4900 1550
+F 0 "#PWR?" H 4900 1400 50  0001 C CNN
+F 1 "+5V" H 4915 1723 50  0000 C CNN
+F 2 "" H 4900 1550 50  0001 C CNN
+F 3 "" H 4900 1550 50  0001 C CNN
+	1    4900 1550
+	1    0    0    -1
+$EndComp
+Wire Wire Line
+	4800 2050 4900 2050
+Wire Wire Line
+	4900 1750 4900 2050
+Connection ~ 4900 2050
+Wire Wire Line
+	4900 2050 5000 2050
 $EndSCHEMATC

Commit message: USB and ISP wiring
Parts:
- added D?: 1N4148, symbol Device:D_Small
- added D? (x2): 3,6 V, symbol Device:D_Zener_Small
- added F1: 500 mA, symbol Device:Polyfuse_Small
- added J1: AVR-ISP-6, symbol Connector:AVR-ISP-6
- added MX?: MX-NoLED, symbol MX_Alps_Hybrid:MX-NoLED
- added R2, R3: 22R, symbol Device:R_Small
- added SW2: BOOT, symbol Switch:SW_Push
- added USB1: Molex-0548190589, symbol random-keyboard-parts:Molex-0548190589
Connections:
- net +5V: now also F1.1, J1.2 (VCC)
- net GND: now also D?.2 (A), D?.2 (A), J1.6 (GND), SW2.2, USB1.1 (GND)
- net at U1.16 (PD2): now also R2.2
- net at U1.17 (PD3): now also R3.2
- net at U1.18 (PD4): now also SW2.1
- net MOSI: now reaches U1.6 (PB5)
- net MOSI: now also J1.4 (MOSI)
- net MISO: now reaches U1.7 (PB6)
- net MISO: now also J1.1 (MISO)
- net SCK: now reaches U1.8 (PB7)
- net SCK: now also J1.3 (SCK)
- net RST: now reaches R1.2, SW1.2, U1.9 (~RESET)
- net RST: now also J1.5 (~RST)
- new net: D?.2 (A), MX?.2 (ROW)
- new net D+: D?.1 (K), R2.1, USB1.3 (D+)
- new net D-: D?.1 (K), R3.1, USB1.4 (D-)
- new net VCC: F1.2, USB1.5 (VBUS)
Other:
- moved on the sheet: C1, C2, C3, C4, C5, R1, SW1, U1, Y1

Commit message: added matrix
Parts:
- added D10, D11, D12, D13, D14, D15, D16, D17, D18, D19, D2, D20, D21, D22, D23, D24, D25, D26, D27, D28, D29, D3, D30, D31, D32, D33, D34, D35, D36, D37, D38, D39, D4, D40, D41, D42, D43, D44, D45, D46, D47, D5, D6, D7, D8, D9: 1N4148, symbol Device:D_Small
- added D50, D51, D52, D53, D54, D55, D56, D57, D58, D59, D60, D61, D62, D63, D64, D65: WS2812B, LED_SMD:LED_WS2812B_PLCC4_5.0x5.0mm_P3.2mm, symbol LED:WS2812B
- added MX10, MX11, MX12, MX13, MX14, MX15, MX16, MX17, MX18, MX19, MX2, MX20, MX21, MX22, MX23, MX24, MX25, MX26, MX27, MX28, MX29, MX3, MX30, MX31, MX32, MX33, MX34, MX35, MX36, MX37, MX38, MX39, MX4, MX40, MX41, MX42, MX43, MX44, MX45, MX46, MX47, MX5, MX6, MX7, MX8, MX9: MX-NoLED, symbol MX_Alps_Hybrid:MX-NoLED
- added R4: 470R, symbol Device:R_Small
- gave numbers to parts that had none: 4
- renumbered C3 to C1, C4 to C2, C5 to C3, C1 to C4, C2 to C5
Connections:
- net +5V: now also D50.1 (VDD), D51.1 (VDD), D52.1 (VDD), D53.1 (VDD), D54.1 (VDD), D55.1 (VDD), D56.1 (VDD), D57.1 (VDD), D58.1 (VDD), D59.1 (VDD), D60.1 (VDD), D61.1 (VDD), D62.1 (VDD), D63.1 (VDD), D64.1 (VDD), D65.1 (VDD)
- net GND: now also D50.3 (VSS), D51.3 (VSS), D52.3 (VSS), D53.3 (VSS), D54.3 (VSS), D55.3 (VSS), D56.3 (VSS), D57.3 (VSS), D58.3 (VSS), D59.3 (VSS), D60.3 (VSS), D61.3 (VSS), D62.3 (VSS), D63.3 (VSS), D64.3 (VSS), D65.3 (VSS)
- net COL0: now reaches MX1.1 (COL)
- net COL0: now also MX2.1 (COL), MX3.1 (COL), MX4.1 (COL)
- net ROW0: now reaches D1.1 (K)
- net ROW0: now also D13.1 (K), D17.1 (K), D21.1 (K), D25.1 (K), D28.1 (K), D32.1 (K), D36.1 (K), D40.1 (K), D44.1 (K), D5.1 (K), D9.1 (K)
- new net: D5.2 (A), MX5.2 (ROW)
- new net: D9.2 (A), MX9.2 (ROW)
- new net: D13.2 (A), MX13.2 (ROW)
- new net: D17.2 (A), MX17.2 (ROW)
- new net: D21.2 (A), MX21.2 (ROW)
- new net: D25.2 (A), MX25.2 (ROW)
- new net: D28.2 (A), MX28.2 (ROW)
- new net: D32.2 (A), MX32.2 (ROW)
- new net: D36.2 (A), MX36.2 (ROW)
- new net: D40.2 (A), MX40.2 (ROW)
- new net: D44.2 (A), MX44.2 (ROW)
- new net: D2.2 (A), MX2.2 (ROW)
- new net: D6.2 (A), MX6.2 (ROW)
- new net: D10.2 (A), MX10.2 (ROW)
- new net: D14.2 (A), MX14.2 (ROW)
- new net: D18.2 (A), MX18.2 (ROW)
- new net: D22.2 (A), MX22.2 (ROW)
- new net: D26.2 (A), MX26.2 (ROW)
- new net: D29.2 (A), MX29.2 (ROW)
- new net: D33.2 (A), MX33.2 (ROW)
- new net: D37.2 (A), MX37.2 (ROW)
- new net: D41.2 (A), MX41.2 (ROW)
- new net: D45.2 (A), MX45.2 (ROW)
- new net: D3.2 (A), MX3.2 (ROW)
- new net: D7.2 (A), MX7.2 (ROW)
- new net: D11.2 (A), MX11.2 (ROW)
- new net: D15.2 (A), MX15.2 (ROW)
- new net: D19.2 (A), MX19.2 (ROW)
- new net: D23.2 (A), MX23.2 (ROW)
- new net: D27.2 (A), MX27.2 (ROW)
- new net: D30.2 (A), MX30.2 (ROW)
- new net: D34.2 (A), MX34.2 (ROW)
- new net: D38.2 (A), MX38.2 (ROW)
- new net: D42.2 (A), MX42.2 (ROW)
- new net: D46.2 (A), MX46.2 (ROW)
- new net: D4.2 (A), MX4.2 (ROW)
- new net: D8.2 (A), MX8.2 (ROW)
- new net: D12.2 (A), MX12.2 (ROW)
- new net: D16.2 (A), MX16.2 (ROW)
- new net: D20.2 (A), MX20.2 (ROW)
- new net: D24.2 (A), MX24.2 (ROW)
- new net: D31.2 (A), MX31.2 (ROW)
- new net: D35.2 (A), MX35.2 (ROW)
- new net: D39.2 (A), MX39.2 (ROW)
- new net: D43.2 (A), MX43.2 (ROW)
- new net: D47.2 (A), MX47.2 (ROW)
- new net: D50.2 (DOUT), D51.4 (DIN)
- new net: D50.4 (DIN), R4.1
- new net: D51.2 (DOUT), D52.4 (DIN)
- new net: D52.2 (DOUT), D53.4 (DIN)
- new net: D53.2 (DOUT), D54.4 (DIN)
- new net: D54.2 (DOUT), D55.4 (DIN)
- new net: D55.2 (DOUT), D56.4 (DIN)
- new net: D56.2 (DOUT), D57.4 (DIN)
- new net: D57.2 (DOUT), D58.4 (DIN)
- new net: D58.2 (DOUT), D59.4 (DIN)
- new net: D59.2 (DOUT), D60.4 (DIN)
- new net: D60.2 (DOUT), D61.4 (DIN)
- new net: D61.2 (DOUT), D62.4 (DIN)
- new net: D62.2 (DOUT), D63.4 (DIN)
- new net: D63.2 (DOUT), D64.4 (DIN)
- new net: D64.2 (DOUT), D65.4 (DIN)
- new net COL1: MX5.1 (COL), MX6.1 (COL), MX7.1 (COL), MX8.1 (COL)
- new net COL10: MX40.1 (COL), MX41.1 (COL), MX42.1 (COL), MX43.1 (COL)
- new net COL11: MX44.1 (COL), MX45.1 (COL), MX46.1 (COL), MX47.1 (COL)
- new net COL2: MX10.1 (COL), MX11.1 (COL), MX12.1 (COL), MX9.1 (COL)
- new net COL3: MX13.1 (COL), MX14.1 (COL), MX15.1 (COL), MX16.1 (COL)
- new net COL4: MX17.1 (COL), MX18.1 (COL), MX19.1 (COL), MX20.1 (COL)
- new net COL5: MX21.1 (COL), MX22.1 (COL), MX23.1 (COL), MX24.1 (COL)
- new net COL6: MX25.1 (COL), MX26.1 (COL), MX27.1 (COL)
- new net COL7: MX28.1 (COL), MX29.1 (COL), MX30.1 (COL), MX31.1 (COL)
- new net COL8: MX32.1 (COL), MX33.1 (COL), MX34.1 (COL), MX35.1 (COL)
- new net COL9: MX36.1 (COL), MX37.1 (COL), MX38.1 (COL), MX39.1 (COL)
- new net RGB: R4.2
- new net ROW1: D10.1 (K), D14.1 (K), D18.1 (K), D2.1 (K), D22.1 (K), D26.1 (K), D29.1 (K), D33.1 (K), D37.1 (K), D41.1 (K), D45.1 (K), D6.1 (K)
- new net ROW2: D11.1 (K), D15.1 (K), D19.1 (K), D23.1 (K), D27.1 (K), D3.1 (K), D30.1 (K), D34.1 (K), D38.1 (K), D42.1 (K), D46.1 (K), D7.1 (K)
- new net ROW3: D12.1 (K), D16.1 (K), D20.1 (K), D24.1 (K), D31.1 (K), D35.1 (K), D39.1 (K), D4.1 (K), D43.1 (K), D47.1 (K), D8.1 (K)
Other:
- moved on the sheet: D1, MX1

Commit message: minor adjustments
Connections:
- net D+: now also U1.16 (PD2); no longer D48.1 (K), USB1.3 (D+)
- net D-: now also U1.17 (PD3); no longer D49.1 (K), USB1.4 (D-)
- net at R2.2: now also D48.1 (K), USB1.3 (D+); no longer U1.16 (PD2)
- net at R3.2: now also D49.1 (K), USB1.4 (D-); no longer U1.17 (PD3)
- net SCL: now reaches U1.22 (PC0)
- net SDA: now reaches U1.23 (PC1)
Other:
- moved on the sheet: C1, C2, C3, C4, C5, D48, D49, F1, J1, R1, R2, R3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

Commit message: schema hopefully complete
Parts:
- added OL1: OLED 128x32, symbol kbd:OLED
Connections:
- net +5V: now also OL1.3 (VCC)
- net COL0: now also U1.40 (PA0)
- net COL1: now also U1.39 (PA1)
- net COL10: now also U1.25 (PC3)
- net COL11: now also U1.24 (PC2)
- net COL2: now also U1.38 (PA2)
- net COL3: now also U1.37 (PA3)
- net COL4: now also U1.36 (PA4)
- net COL5: now also U1.35 (PA5)
- net COL6: now also U1.34 (PA6)
- net COL7: now also U1.33 (PA7)
- net COL8: now also U1.27 (PC5)
- net COL9: now also U1.26 (PC4)
- net GND: now also OL1.4 (GND)
- net ROW0: now also U1.1 (PB0)
- net ROW1: now also U1.2 (PB1)
- net ROW2: now also U1.3 (PB2)
- net ROW3: now also U1.4 (PB3)
- net SCL: now also OL1.2 (SCL)
- net SDA: now also OL1.1 (SDA)
Changed lines of the file:
@@
 Wire Wire Line
 	5950 6950 6100 6950
-Text GLabel 2850 1350 2    50   Input ~ 0
+Text GLabel 3250 4600 2    50   Input ~ 0
 ROW0
-Text GLabel 2850 1450 2    50   Input ~ 0
+Text GLabel 3250 4700 2    50   Input ~ 0
 ROW1
-Text GLabel 2850 1550 2    50   Input ~ 0
+Text GLabel 3250 4800 2    50   Input ~ 0
 ROW2
-Text GLabel 2850 1650 2    50   Input ~ 0
+Text GLabel 3250 4900 2    50   Input ~ 0
 ROW3
-Text GLabel 3200 1350 2    50   Input ~ 0
+Text GLabel 3250 3700 2    50   Input ~ 0
 COL0
-Text GLabel 3200 1450 2    50   Input ~ 0
+Text GLabel 3250 3800 2    50   Input ~ 0
 COL1
-Text GLabel 3200 1550 2    50   Input ~ 0
+Text GLabel 3250 3900 2    50   Input ~ 0
 COL2
-Text GLabel 3200 1650 2    50   Input ~ 0
+Text GLabel 3250 4000 2    50   Input ~ 0
 COL3
-Text GLabel 3200 1750 2    50   Input ~ 0
+Text GLabel 3250 4100 2    50   Input ~ 0
 COL4
-Text GLabel 3200 1850 2    50   Input ~ 0
+Text GLabel 3250 4200 2    50   Input ~ 0
 COL5
-Text GLabel 3200 1950 2    50   Input ~ 0
+Text GLabel 3250 4300 2    50   Input ~ 0
 COL6
-Text GLabel 3200 2050 2    50   Input ~ 0
+Text GLabel 3250 4400 2    50   Input ~ 0
 COL7
-Text GLabel 3200 2150 2    50   Input ~ 0
+Text GLabel 3250 6000 2    50   Input ~ 0
 COL8
-Text GLabel 3200 2250 2    50   Input ~ 0
+Text GLabel 3250 5900 2    50   Input ~ 0
 COL9
-Text GLabel 3200 2350 2    50   Input ~ 0
+Text GLabel 3250 5800 2    50   Input ~ 0
 COL10
-Text GLabel 3200 2450 2    50   Input ~ 0
+Text GLabel 3250 5700 2    50   Input ~ 0
 COL11
 Text GLabel 2850 2150 2    50   Input ~ 0
@@
 Text GLabel 3250 5600 2    50   Input ~ 0
 SDA
+$Comp
+L kbd:OLED OL1
+U 1 1 615D634B
+P 2050 1100
+F 0 "OL1" H 2678 1169 51  0000 L CNN
+F 1 "OLED 128x32" H 2678 1079 47  0000 L CNN
+F 2 "" H 2050 1200 60  0001 C CNN
+F 3 "" H 2050 1200 60  0001 C CNN
+	1    2050 1100
+	1    0    0    -1
+$EndComp
+Text GLabel 1300 1000 0    50   Input ~ 0
+SCL
+Text GLabel 1300 850  0    50   Input ~ 0
+SDA
+$Comp
+L power:+5V #PWR?
+U 1 1 615D9D0C
+P 950 1150
+F 0 "#PWR?" H 950 1000 50  0001 C CNN
+F 1 "+5V" H 965 1323 50  0000 C CNN
+F 2 "" H 950 1150 50  0001 C CNN
+F 3 "" H 950 1150 50  0001 C CNN
+	1    950  1150
+	1    0    0    -1
+$EndComp
+Wire Wire Line
+	950  1150 1300 1150
+$Comp
+L power:GND #PWR?
+U 1 1 615EB060
+P 950 1300
+F 0 "#PWR?" H 950 1050 50  0001 C CNN
+F 1 "GND" H 955 1127 50  0000 C CNN
+F 2 "" H 950 1300 50  0001 C CNN
+F 3 "" H 950 1300 50  0001 C CNN
+	1    950  1300
+	1    0    0    -1
+$EndComp
+Wire Wire Line
+	950  1300 1300 1300
 $EndSCHEMATC
